File: HW/RTL/06PCM-AUDIO-MICROFONO/Version_01/04 PCB/Microfono/Microfono.kicad_pcb (KiCad board)
At the start: 2 copper layers, 9 parts, among them J1 CONN_01X05

Commit message: act kicad
Parts:
- C1, C2: value CP1_Small -> 0.1uF; footprint Capacitors_Tantalum_SMD:CP_Tantalum_Case-A_EIA-3216-18_Hand -> Resistors_SMD:R_0805_HandSoldering
- C3, C4: value CP1_Small -> 200pf; footprint Capacitors_Tantalum_SMD:CP_Tantalum_Case-A_EIA-3216-18_Hand -> Capacitors_SMD:C_0805_HandSoldering
- MK1, MK2: footprint MIC_SPH0645LM4H-B -> microfono:MIC_SPH0645LM4H-B
- R1, R2: value R_Small -> R; footprint Resistors_SMD:R_0201 -> Resistors_SMD:R_0805
Connections:
- net Net-(C1-Pad1) renamed VCC
- net Net-(J1-Pad4) renamed /data
- C2 pad 2: Net-(C1-Pad2) -> Net-(C2-Pad2)
- C4 pad 2: Net-(C1-Pad2) -> Net-(C2-Pad2)
- J1 pad 2: Net-(C1-Pad2) -> /ws
- J1 pad 3: Net-(J1-Pad3) -> /bclk
- J1 pad 5: Net-(J1-Pad5) -> GND
- MK1 pad 1: Net-(J1-Pad3) -> /ws
- MK1 pad 3: Net-(C1-Pad2) -> GND
- MK1 pad 4: Net-(J1-Pad5) -> /bclk
- MK2 pad 1: Net-(J1-Pad3) -> /ws
- MK2 pad 2: Net-(C1-Pad2) -> GND
- MK2 pad 3: Net-(C1-Pad2) -> GND
- MK2 pad 4: Net-(J1-Pad5) -> /bclk
- R1 pad 2: Net-(MK2-Pad6) -> Net-(MK1-Pad6)
- R2 pad 2: Net-(MK1-Pad6) -> Net-(MK2-Pad6)
Routing:
- net Net-(C1-Pad2): track 48.5 -> 16.3 mm
- net Net-(J1-Pad5): track 15.1 -> 0.00 mm
- net Net-(J1-Pad3): track 13.7 -> 0.00 mm
