File: HW/RTL/06PCM-AUDIO-MICROFONO/Version_01/04 PCB/Microfono/Microfono.sch (KiCad schematic (older format))
At the start: 9 parts, among them J1 CONN_01X05

Commit message: act kicad
Parts:
- removed C1, C2, C3, C4: CP1_Small, Capacitors_Tantalum_SMD:CP_Tantalum_Case-A_EIA-3216-18_Hand, symbol CP1_Small
- removed MK2: SPH0645LM4H-B, SPH0645LM4H-B:MIC_SPH0645LM4H-B, symbol SPH0645LM4H-B
- removed R1, R2: R_Small, Resistors_SMD:R_0201, symbol R_Small
- added C? (x2): 0.1uF, Resistors_SMD:R_0805_HandSoldering, symbol C
- added C? (x2): 200pf, Capacitors_SMD:C_0805_HandSoldering, symbol C
- added MK?: SPH0645LM4H-B, microfono:MIC_SPH0645LM4H-B, symbol SPH0645LM4H-B
- added R? (x2): R, Resistors_SMD:R_0805, symbol R
- MK1: footprint SPH0645LM4H-B:MIC_SPH0645LM4H-B -> microfono:MIC_SPH0645LM4H-B
Connections:
- net labels added: GND, VCC, bclk, data, ws
- wire segments 45 -> 30
Other:
- moved on the sheet: J1, MK1

Commit message: carpeta
Parts:
- gave numbers to parts that had none: 7
Changed lines of the file:
@@
 $EndComp
 $Comp
-L C C?
+L C C1
 U 1 1 59AEF705
 P 5900 3150
-F 0 "C?" H 5925 3250 50  0000 L CNN
+F 0 "C1" H 5925 3250 50  0000 L CNN
 F 1 "0.1uF" H 5925 3050 50  0000 L CNN
 F 2 "Resistors_SMD:R_0805_HandSoldering" H 5938 3000 50  0001 C CNN
@@
 $EndComp
 $Comp
-L C C?
+L C C3
 U 1 1 59AEF871
 P 6200 3150
-F 0 "C?" H 6225 3250 50  0000 L CNN
+F 0 "C3" H 6225 3250 50  0000 L CNN
 F 1 "200pf" H 6225 3050 50  0000 L CNN
 F 2 "Capacitors_SMD:C_0805_HandSoldering" H 6238 3000 50  0001 C CNN
@@
 $EndComp
 $Comp
-L GND #PWR01
+L GND #PWR6
 U 1 1 59AEFF91
 P 6550 4050
-F 0 "#PWR01" H 6550 3800 50  0001 C CNN
+F 0 "#PWR6" H 6550 3800 50  0001 C CNN
 F 1 "GND" H 6550 3900 50  0000 C CNN
 F 2 "" H 6550 4050 50  0001 C CNN
@@
 $EndComp
 $Comp
-L VCC #PWR02
+L VCC #PWR5
 U 1 1 59AEFFBD
 P 6550 2900
-F 0 "#PWR02" H 6550 2750 50  0001 C CNN
+F 0 "#PWR5" H 6550 2750 50  0001 C CNN
 F 1 "VCC" H 6550 3050 50  0000 C CNN
 F 2 "" H 6550 2900 50  0001 C CNN
@@
 $EndComp
 $Comp
-L GND #PWR03
+L GND #PWR3
 U 1 1 59AF03CA
 P 6050 3300
-F 0 "#PWR03" H 6050 3050 50  0001 C CNN
+F 0 "#PWR3" H 6050 3050 50  0001 C CNN
 F 1 "GND" H 6050 3150 50  0000 C CNN
 F 2 "" H 6050 3300 50  0001 C CNN
@@
 $EndComp
 $Comp
-L VCC #PWR04
+L VCC #PWR1
 U 1 1 59AF06A9
 P 4800 3750
-F 0 "#PWR04" H 4800 3600 50  0001 C CNN
+F 0 "#PWR1" H 4800 3600 50  0001 C CNN
 F 1 "VCC" H 4800 3900 50  0000 C CNN
 F 2 "" H 4800 3750 50  0001 C CNN
@@
 $EndComp
 $Comp
-L R R?
+L R R1
 U 1 1 59AF08CC
 P 6800 3800
-F 0 "R?" V 6880 3800 50  0000 C CNN
+F 0 "R1" V 6880 3800 50  0000 C CNN
 F 1 "R" V 6800 3800 50  0000 C CNN
 F 2 "Resistors_SMD:R_0805" V 6730 3800 50  0001 C CNN
@@
 data
 $Comp
-L VCC #PWR05
+L VCC #PWR10
 U 1 1 59AF0D15
 P 7900 4250
-F 0 "#PWR05" H 7900 4100 50  0001 C CNN
+F 0 "#PWR10" H 7900 4100 50  0001 C CNN
 F 1 "VCC" H 7900 4400 50  0000 C CNN
 F 2 "" H 7900 4250 50  0001 C CNN
@@
 data
 $Comp
-L GND #PWR06
+L GND #PWR9
 U 1 1 59AF0EA3
 P 7850 4700
-F 0 "#PWR06" H 7850 4450 50  0001 C CNN
+F 0 "#PWR9" H 7850 4450 50  0001 C CNN
 F 1 "GND" H 7850 4550 50  0000 C CNN
 F 2 "" H 7850 4700 50  0001 C CNN
@@
 $EndComp
 $Comp
-L SPH0645LM4H-B MK?
+L SPH0645LM4H-B MK2
 U 1 1 59AEFDA3
 P 5800 5750
-F 0 "MK?" H 5299 5971 50  0000 L BNN
+F 0 "MK2" H 5299 5971 50  0000 L BNN
 F 1 "SPH0645LM4H-B" H 5299 5450 50  0000 L BNN
 F 2 "microfono:MIC_SPH0645LM4H-B" H 5800 5750 50  0001 L BNN
@@
 $EndComp
 $Comp
-L C C?
+L C C2
 U 1 1 59AEFDAA
 P 5900 5100
-F 0 "C?" H 5925 5200 50  0000 L CNN
+F 0 "C2" H 5925 5200 50  0000 L CNN
 F 1 "0.1uF" H 5925 5000 50  0000 L CNN
 F 2 "Resistors_SMD:R_0805_HandSoldering" H 5938 4950 50  0001 C CNN
@@
 $EndComp
 $Comp
-L C C?
+L C C4
 U 1 1 59AEFDB1
 P 6200 5100
-F 0 "C?" H 6225 5200 50  0000 L CNN
+F 0 "C4" H 6225 5200 50  0000 L CNN
 F 1 "200pf" H 6225 5000 50  0000 L CNN
 F 2 "Capacitors_SMD:C_0805_HandSoldering" H 6238 4950 50  0001 C CNN
@@
 $EndComp
 $Comp
-L GND #PWR?
+L GND #PWR8
 U 1 1 59AEFDB8
 P 6550 6000
-F 0 "#PWR?" H 6550 5750 50  0001 C CNN
+F 0 "#PWR8" H 6550 5750 50  0001 C CNN
 F 1 "GND" H 6550 5850 50  0000 C CNN
 F 2 "" H 6550 6000 50  0001 C CNN
@@
 $EndComp
 $Comp
-L VCC #PWR?
+L VCC #PWR7
 U 1 1 59AEFDBE
 P 6550 4850
-F 0 "#PWR?" H 6550 4700 50  0001 C CNN
+F 0 "#PWR7" H 6550 4700 50  0001 C CNN
 F 1 "VCC" H 6550 5000 50  0000 C CNN
 F 2 "" H 6550 4850 50  0001 C CNN
@@
 $EndComp
 $Comp
-L GND #PWR?
+L GND #PWR4
 U 1 1 59AEFDC4
 P 6050 5250
-F 0 "#PWR?" H 6050 5000 50  0001 C CNN
+F 0 "#PWR4" H 6050 5000 50  0001 C CNN
 F 1 "GND" H 6050 5100 50  0000 C CNN
 F 2 "" H 6050 5250 50  0001 C CNN
@@
 $EndComp
 $Comp
-L R R?
+L R R2
 U 1 1 59AEFDD0
 P 6800 5750
-F 0 "R?" V 6880 5750 50  0000 C CNN
+F 0 "R2" V 6880 5750 50  0000 C CNN
 F 1 "R" V 6800 5750 50  0000 C CNN
 F 2 "Resistors_SMD:R_0805" V 6730 5750 50  0001 C CNN
@@
 data
 $Comp
-L GND #PWR?
+L GND #PWR2
 U 1 1 59AEFE5D
 P 4800 5900
-F 0 "#PWR?" H 4800 5650 50  0001 C CNN
+F 0 "#PWR2" H 4800 5650 50  0001 C CNN
 F 1 "GND" H 4800 5750 50  0000 C CNN
 F 2 "" H 4800 5900 50  0001 C CNN
